File: PCB/LED-Board-MW/LED-Board-MW.sch (KiCad schematic (older format))
At the start: 23 parts, among them T1 1755736, T2 1755736, T3 1755736, U1 TPS61165DBVR, U2 TPS61165DBVR

Commit message: Board Started
Started doing board based on schetaic, design make change since LEDs are huge
Parts:
- C7, C8: footprint AVR-KiCAD-Lib-Diodes:D_SOD-123 -> AVR-KiCAD-Lib-Capacitors:C1206
Changed lines of the file:
@@
 F 0 "C7" V 9829 2178 50  0000 L CNN
 F 1 "C1206C105K3RACAUTO" H 9900 2250 50  0001 C CNN
-F 2 "AVR-KiCAD-Lib-Diodes:D_SOD-123" H 9650 2050 50  0001 C CNN
+F 2 "AVR-KiCAD-Lib-Capacitors:C1206" H 9650 2050 50  0001 C CNN
 F 3 "https://content.kemet.com/datasheets/KEM_C1023_X7R_AUTO_SMD.pdf" H 9750 2150 50  0001 C CNN
 F 4 "0.25000" H 9950 2300 50  0001 C CNN "Cost QTY: 1"
@@
 F 0 "C8" V 9829 4278 50  0000 L CNN
 F 1 "C1206C105K3RACAUTO" H 9900 4350 50  0001 C CNN
-F 2 "AVR-KiCAD-Lib-Diodes:D_SOD-123" H 9650 4150 50  0001 C CNN
+F 2 "AVR-KiCAD-Lib-Capacitors:C1206" H 9650 4150 50  0001 C CNN
 F 3 "https://content.kemet.com/datasheets/KEM_C1023_X7R_AUTO_SMD.pdf" H 9750 4250 50  0001 C CNN
 F 4 "0.25000" H 9950 4400 50  0001 C CNN "Cost QTY: 1"
